File: Base/White Mount/Pololu Magnetic Encoder Base.brd (EAGLE design)
At the start: 26.7 x 33.7 mm, 0 parts

Commit message: Messing with encoders. Created base plate for Black Mount Created two PCBs for base-less/floating encoder
Other:
- board text added: "AnomalousMaker.com"
- board text removed: "innovativemaker.com"
Changed lines of the file:
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@@
 <?xml version="1.0" encoding="utf-8"?>
 <!DOCTYPE eagle SYSTEM "eagle.dtd">
-<eagle version="6.3">
+<eagle version="6.4">
 <drawing>
 <settings>
@@
 <hole x="8.89" y="31.3055" drill="1.6"/>
 <hole x="19.05" y="31.3055" drill="1.6"/>
-<text x="8.255" y="22.86" size="1.778" layer="51" font="vector" ratio="12">3.3v</text>
-<text x="8.255" y="20.32" size="1.778" layer="51" font="vector" ratio="12">GND</text>
-<text x="18.415" y="22.86" size="1.778" layer="51" font="vector" ratio="12">A</text>
-<text x="18.415" y="20.32" size="1.778" layer="51" font="vector" ratio="12">B</text>
-<text x="13.335" y="22.86" size="1.778" layer="52" font="vector" ratio="12" rot="MR0">3.3v</text>
-<text x="13.335" y="20.32" size="1.778" layer="52" font="vector" ratio="12" rot="MR0">GND</text>
-<text x="19.685" y="20.32" size="1.778" layer="52" font="vector" ratio="12" rot="MR0">B</text>
-<text x="19.685" y="22.86" size="1.778" layer="52" font="vector" ratio="12" rot="MR0">A</text>
+<text x="8.255" y="26.67" size="1.778" layer="51" font="vector" ratio="12">3.3v</text>
+<text x="8.255" y="24.13" size="1.778" layer="51" font="vector" ratio="12">GND</text>
+<text x="18.415" y="26.67" size="1.778" layer="51" font="vector" ratio="12">A</text>
+<text x="18.415" y="24.13" size="1.778" layer="51" font="vector" ratio="12">B</text>
+<text x="13.335" y="26.67" size="1.778" layer="52" font="vector" ratio="12" rot="MR0">3.3v</text>
+<text x="13.335" y="24.13" size="1.778" layer="52" font="vector" ratio="12" rot="MR0">GND</text>
+<text x="19.685" y="24.13" size="1.778" layer="52" font="vector" ratio="12" rot="MR0">B</text>
+<text x="19.685" y="26.67" size="1.778" layer="52" font="vector" ratio="12" rot="MR0">A</text>
 <wire x1="5.08" y1="17.78" x2="5.08" y2="8.89" width="0" layer="20" curve="180"/>
 <wire x1="22.86" y1="17.78" x2="22.86" y2="8.89" width="0" layer="20" curve="-180"/>
@@
 <rectangle x1="9.525" y1="29.21" x2="18.415" y2="30.48" layer="29" rot="R180"/>
 <text x="13.97" y="1.905" size="0.8128" layer="52" font="vector" ratio="12" rot="MR0" align="bottom-center">Cruz Monrreal II</text>
-<text x="13.97" y="0.635" size="0.8128" layer="52" font="vector" ratio="12" rot="MR0" align="bottom-center">innovativemaker.com</text>
+<text x="13.97" y="0.635" size="0.8128" layer="52" font="vector" ratio="12" rot="MR0" align="bottom-center">AnomalousMaker.com</text>
 </plain>
 <attributes>
