File: Floating/AS5035/Pololu Magnetic Encoder (Floating) (AS5035).brd (EAGLE design)
At the start: 12 x 12.1 mm, 6 parts, among them U1 AS5035

Commit message: Merge branch 'master' of github.com:cmonr/Other-PCBs
Conflicts:
	TI/Robotics Booster Pack/Robotics Booster Pack.sch
Parts:
- U$5: value 1X7 -> 1X6; device headers(.05in):1X7 -> headers(2mm):1X6
- moved U$5 3.46 mm to (6.00, 11.0)
- moved C1 0.56 mm to (2.54, 6.35), turned to 180 degrees
- moved J1 0.54 mm to (2.54, 4.45)
- moved C2 0.46 mm to (2.54, 2.54)
Connections:
- net NDX: no longer U$5.7
Routing:
- net NDX: track 6.89 -> 0.00 mm
- net N$4: track 6.32 -> 5.01 mm
- net VIN: track 13.8 -> 12.7 mm
Other:
- board text added: "Floating QEI Mag Encoder"
- board text removed: "Floating QEI Mag Enc"
- board text removed: "NDX"
